File: bp-backup/chavdai40-bp-2020-05-16-15-11.kicad_pcb (KiCad board)
At the start: 2 copper layers, 282.6 x 92 mm, 111 parts, among them J1 Conn_ARM_JTAG_SWD_10, U1 STM32F042K6U6, U2 XC6206P332MR

Commit message: tabun dekita
Other:
- outline, holes or cut-outs redrawn
