File: chavdai40.kicad_pcb (KiCad board)
At the start: 2 copper layers, 282.6 x 92 mm, 111 parts, among them J1 Conn_ARM_JTAG_SWD_10, U1 STM32F042K6U6, U2 XC6206P332MR

Commit message: create info.json
Parts:
- D1, D10, D11, D12, D13, D14, D15, D16, D17, D18, D19, D2, D20, D21, D22, D23, D24, D25, D26, D27, D28, D29, D3, D30, D31, D32, D33, D34, D35, D36, D37, D38, D39, D4, D40, D41, D42, D43, D44, D5, D6, D7, D8, D9: footprint Diode_SMD:D_SOD-323F -> Diode_SMD:D_SOD-123
- moved D14 35.0 mm to (70.7, 46.7)
- moved D44 14.2 mm to (240.0, 83.9)
- moved D13 14.0 mm to (264.0, 26.9)
- moved D41 8.62 mm to (170.6, 82.9)
- moved D1 6.44 mm to (27.4, 25.5)
- moved D15 5.79 mm to (74.1, 45.8)
- moved D36 3.11 mm to (254.7, 65.0)
- moved D24 3.08 mm to (242.8, 45.9)
- moved D20 3.08 mm to (166.6, 45.9)
- moved D19 3.00 mm to (147.4, 46.0)
- moved D16 2.96 mm to (90.2, 45.9)
- moved D22 2.96 mm to (204.5, 45.9)
- moved D35 2.96 mm to (233.1, 65.0)
- moved D17 2.96 mm to (109.3, 45.9)
- moved D34 2.96 mm to (214.1, 65.0)
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Routing:
- net ROW1: track 337.5 -> 277.2 mm, vias 2 -> 0
- net ROW0: track 384.4 -> 340.7 mm
- net ROW2: track 399.2 -> 363.5 mm
- net Net-(D14-Pad2): track 3.51 -> 34.9 mm, vias 0 -> 1
- net COL12: track 267.6 -> 239.6 mm
- net ROW3: track 307.9 -> 294.0 mm
- net Net-(D1-Pad2): track 3.21 -> 11.9 mm
- net Net-(D13-Pad2): track 3.22 -> 11.3 mm
- net Net-(D44-Pad2): track 3.22 -> 11.3 mm
- net Net-(D15-Pad2): track 3.22 -> 9.05 mm
- net Net-(D41-Pad2): track 9.78 -> 15.2 mm
- net GND: track 181.6 -> 184.9 mm
- net Net-(D36-Pad2): track 3.22 -> 6.34 mm
- net Net-(D20-Pad2): track 3.22 -> 6.31 mm
- net Net-(D19-Pad2): track 3.22 -> 6.23 mm
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