File: chavdai40.kicad_pcb (KiCad board)
At the start: 2 copper layers, 282.6 x 92 mm, 111 parts, among them J1 Conn_ARM_JTAG_SWD_10, U1 STM32F042K6U6, U2 XC6206P332MR

Commit message: update chavdai pcb design(rev2)
Parts:
- removed SMT1, SMT2, SMT3: Tooling Hole, random-keyboard-parts:jlcpcb-tooling-hole
- added J2: Conn_01x03, Connector_PinHeader_2.54mm:PinHeader_1x03_P2.54mm_Vertical, F.Cu at (34.0, 57.5)
- J1: value Conn_ARM_JTAG_SWD_10 -> Conn_01x02; footprint Connector_PinHeader_1.27mm:PinHeader_2x05_P1.27mm_Vertical -> Connector_PinHeader_2.54mm:PinHeader_1x02_P2.54mm_Vertical
- U1: value STM32F042K6U6 -> STM32F042K6T6; footprint Package_DFN_QFN:QFN-32-1EP_5x5mm_P0.5mm_EP3.45x3.45mm -> Package_QFP:LQFP-32_7x7mm_P0.8mm
- moved D1 38.6 mm to (65.9, 26.8)
- moved D25 23.5 mm to (259.5, 65.0)
- moved D24 19.9 mm to (236.9, 65.0)
- moved C3 4.64 mm to (54.4, 39.9), turned to 180 degrees
- moved J1 3.13 mm to (36.6, 60.1), turned to 270 degrees
- moved D2 2.86 mm to (69.1, 26.8)
- moved C2 1.87 mm to (41.7, 45.3)
- moved C1 1.60 mm to (43.6, 50.0)
- moved U1 1.59 mm to (49.6, 45.1)
- moved C5 0.59 mm to (31.1, 43.1)
Connections:
- J1 pad 1: +3V3 -> GND
- J1 pad 2: SWDIO -> +3V3
- U1 pad 16: COL3 -> GND
- U1 pad 18: Net-(U1-Pad18) -> COL3
- U1 pad 30: Net-(U1-Pad30) -> COL0
- U1 pad 32: COL0 -> GND
Routing:
- net GND: track 184.9 -> 157.7 mm, vias 12 -> 7
- net Net-(D25-Pad2): track 3.57 -> 30.7 mm
- net Net-(D1-Pad2): track 11.9 -> 36.2 mm, vias 0 -> 1
- net ROW0: track 340.7 -> 316.6 mm, vias 2 -> 0
- net Net-(D24-Pad2): track 6.18 -> 25.6 mm, vias 0 -> 1
- net Net-(D14-Pad2): track 34.9 -> 49.4 mm, vias 1 -> 2
- net +3V3: track 87.8 -> 97.9 mm
- net ROW1: track 277.2 -> 284.6 mm
- net Net-(D2-Pad2): track 5.81 -> 10.6 mm
- net NRST: track 38.5 -> 33.8 mm
- net COL3: track 117.2 -> 113.4 mm
- net SWCLK: track 26.2 -> 29.2 mm
- net SWDIO: track 27.4 -> 24.8 mm
- net COL4: track 115.1 -> 113.2 mm
- net COL5: track 167.6 -> 165.9 mm
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- added copper zone on B.Cu, net GND
Other:
- board text added: "3v"
- board text added: "CLK"
- board text added: "DIO"
- board text added: "GND"
- board text added: "NRST"
- board text added: "rev2"
