File: chavdai40-bp.kicad_pcb (KiCad board)
At the start: 2 copper layers, 282.6 x 92 mm, 0 parts

Commit message: update chavdai pcb design(rev2)
Parts:
- added REF**: PinHeader_1x01_P2.54mm_Vertical, Connector_PinHeader_2.54mm:PinHeader_1x01_P2.54mm_Vertical, F.Cu at (290.0, 17.0)
Other:
- outline, holes or cut-outs redrawn
Changed lines of the file:
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@@
   (general
     (thickness 1.6)
-    (drawings 106)
+    (drawings 114)
     (tracks 0)
     (zones 0)
-    (modules 0)
+    (modules 1)
     (nets 1)
   )
@@
       (drillshape 0)
       (scaleselection 1)
-      (outputdirectory "gerbers-bp/"))
+      (outputdirectory "../../Keyboard開発関連/chavdai-jlcpcb-smt/gerbers-bp-v2/"))
   )
   (net 0 "")
@@
     (uvia_drill 0.1)
   )
+  (module Connector_PinHeader_2.54mm:PinHeader_1x01_P2.54mm_Vertical (layer F.Cu)
+    (at 290 17)
+    (descr "Through hole straight pin header, 1x01, 2.54mm pitch, single row")
+    (tags "Through hole pin header THT 1x01 2.54mm single row")
+    (fp_text reference REF** (at 0 -2.33) (layer F.SilkS) hide
+      (effects (font (size 1 1) (thickness 0.15)))
+    )
+    (fp_text value PinHeader_1x01_P2.54mm_Vertical (at 0 2.33) (layer F.Fab)
+      (effects (font (size 1 1) (thickness 0.15)))
+    )
+    (fp_text user %R (at 0 0 90) (layer F.Fab)
+      (effects (font (size 1 1) (thickness 0.15)))
+    )
+    (fp_line (start 1.8 -1.8) (end -1.8 -1.8) (layer F.CrtYd) (width 0.05))
+    (fp_line (start 1.8 1.8) (end 1.8 -1.8) (layer F.CrtYd) (width 0.05))
+    (fp_line (start -1.8 1.8) (end 1.8 1.8) (layer F.CrtYd) (width 0.05))
+    (fp_line (start -1.8 -1.8) (end -1.8 1.8) (layer F.CrtYd) (width 0.05))
+    (fp_line (start -1.33 -1.33) (end 0 -1.33) (layer F.SilkS) (width 0.12))
+    (fp_line (start -1.33 0) (end -1.33 -1.33) (layer F.SilkS) (width 0.12))
+    (fp_line (start -1.33 1.27) (end 1.33 1.27) (layer F.SilkS) (width 0.12))
+    (fp_line (start 1.33 1.27) (end 1.33 1.33) (layer F.SilkS) (width 0.12))
+    (fp_line (start -1.33 1.27) (end -1.33 1.33) (layer F.SilkS) (width 0.12))
+    (fp_line (start -1.33 1.33) (end 1.33 1.33) (layer F.SilkS) (width 0.12))
+    (fp_line (start -1.27 -0.635) (end -0.635 -1.27) (layer F.Fab) (width 0.1))
+    (fp_line (start -1.27 1.27) (end -1.27 -0.635) (layer F.Fab) (width 0.1))
+    (fp_line (start 1.27 1.27) (end -1.27 1.27) (layer F.Fab) (width 0.1))
+    (fp_line (start 1.27 -1.27) (end 1.27 1.27) (layer F.Fab) (width 0.1))
+    (fp_line (start -0.635 -1.27) (end 1.27 -1.27) (layer F.Fab) (width 0.1))
+    (pad 1 thru_hole rect (at 0 0) (size 1.7 1.7) (drill 1) (layers *.Cu *.Mask))
+    (model ${KISYS3DMOD}/Connector_PinHeader_2.54mm.3dshapes/PinHeader_1x01_P2.54mm_Vertical.wrl
+      (at (xyz 0 0 0))
+      (scale (xyz 1 1 1))
+      (rotate (xyz 0 0 0))
+    )
+  )
+  (gr_line (start 42.7 41.7) (end 27.6 41.7) (layer Edge.Cuts) (width 0.05))
+  (gr_line (start 44.3 39) (end 56.2 39) (layer Edge.Cuts) (width 0.05))
+  (gr_arc (start 42.7 40.9) (end 43.5 40.9) (angle 90) (layer Edge.Cuts) (width 0.05))
+  (gr_line (start 43.5 39.8) (end 43.5 40.9) (layer Edge.Cuts) (width 0.05))
+  (gr_arc (start 44.3 39.8) (end 43.5 39.8) (angle 90) (layer Edge.Cuts) (width 0.05))
+  (gr_line (start 57 39.8) (end 57 40.9) (layer Edge.Cuts) (width 0.05))
+  (gr_arc (start 56.2 39.8) (end 57 39.8) (angle -90) (layer Edge.Cuts) (width 0.05))
+  (gr_arc (start 57.8 40.9) (end 57 40.9) (angle -90) (layer Edge.Cuts) (width 0.05))
   (gr_text JLCJLCJLCJLC (at 160.082 56.323) (layer F.SilkS)
     (effects (font (size 1 1) (thickness 0.15)))
   )
-  (gr_line (start 239.6 41.7) (end 27.6 41.7) (layer Edge.Cuts) (width 0.05))
+  (gr_line (start 239.6 41.7) (end 57.8 41.7) (layer Edge.Cuts) (width 0.05))
   (gr_line (start 241.6 43.7) (end 241.6 49) (layer Edge.Cuts) (width 0.05))
   (gr_arc (start 239.6 49) (end 239.6 51) (angle -90) (layer Edge.Cuts) (width 0.05))
